Commit message: Fix robot model, inflation-escape replan, live-editable dimensions
- Move laser_link from front-edge (x=0.15) to chassis-center (x=0.01)
  matching the physical mount, and drive base_link→laser_link from
  robot_state_publisher instead of a 0,0,0 static_tf override
- Add robot.urdf.xacro + build_urdf.py renderer; launches merge in
  ~/.autonexa/robot_dimensions.yaml and feed the matching footprint
  to both Nav2 costmaps
- Wrap send_nav_goal with an inflation-escape sequence (clear costmaps,
  inflation_radius → 0.01 m, restore on first /plan or 4 s) so SMAC
  Hybrid-A* can plan from a wall-parked start
- Enable bt_navigate_to_pose_ackermann.xml (1 Hz periodic replan +
  ClearCostmap/BackUp recoveries) so the planner recovers when
  collision_monitor stalls a still-valid path
- collision_monitor.time_before_collision 1.2 → 0.9 s;
  min_lookahead_dist 0.16 → 0.14
- New /api/robot_config endpoint regenerates URDF, SetParameters on
  /robot_state_publisher + both costmaps, persists to disk
- App: render chassis footprint + red LiDAR marker on the map tab;
  new Settings → Robot Dimensions dialog with live preview
- RViz: add RobotModel display to navigation.rviz; flip visualization
  .rviz description-topic durability volatile → transient local

Co-Authored-By: Claude Opus 4.7 (1M context) <noreply@anthropic.com>

File: src/parking_system/urdf/robot.urdf.xacro (robot description, xacro)
@@ -1,9 +1,12 @@
 <?xml version="1.0"?>
 <!--
-  Static fallback URDF. The authoritative source is robot.urdf.xacro plus
-  ~/.autonexa/robot_dimensions.yaml, rendered by scripts/build_urdf.py at
-  launch time and live-edited by the mobile bridge. This file is kept in
-  sync with the xacro defaults so any tool that still reads robot.urdf
-  directly gets the corrected geometry.
+  AutoNexa robot description — template form.
+  Substitution happens in scripts/parking_system/build_urdf.py (pure-Python,
+  no `xacro` subprocess). Each brace-delimited token below is replaced with a
+  numeric value coming from defaults + ~/.autonexa/robot_dimensions.yaml +
+  any in-flight override from the mobile bridge.
+  Coordinate frames are right-handed: x forward, y left, z up; base_link is
+  at the chassis geometric center on the ground plane (z=0 here, no wheel
+  links yet so the chassis box just hovers).
 -->
 <robot name="parking_robot">
@@ -11,5 +14,5 @@
     <visual>
       <geometry>
-        <box size="0.3 0.2 0.1"/>
+        <box size="{chassis_length} {chassis_width} {chassis_height}"/>
       </geometry>
       <material name="base_color">
@@ -19,5 +22,5 @@
     <collision>
       <geometry>
-        <box size="0.3 0.2 0.1"/>
+        <box size="{chassis_length} {chassis_width} {chassis_height}"/>
       </geometry>
     </collision>
@@ -41,8 +44,14 @@
     </inertial>
   </link>
+  <!--
+    LiDAR is physically mounted with its cable / 0° marker pointing
+    backwards; yaw = π reconciles that so scan rays resolve correctly in
+    base_link frame. The XYZ offset is the puck's rotation axis relative to
+    the chassis geometric center.
+  -->
   <joint name="laser_joint" type="fixed">
     <parent link="base_link"/>
     <child link="laser_link"/>
-    <origin xyz="0.01 0.0 0.07" rpy="0 0 3.14159"/>
+    <origin xyz="{lidar_x} {lidar_y} {lidar_z}" rpy="0 0 3.14159"/>
   </joint>
   <link name="camera_link">
@@ -63,5 +72,5 @@
     <parent link="base_link"/>
     <child link="camera_link"/>
-    <origin xyz="0.1 0.0 0.05" rpy="0 0 0"/>
+    <origin xyz="{camera_x} 0.0 {camera_z}" rpy="0 0 0"/>
   </joint>
 </robot>
