Commit message: Fix scan-walls mismatch + Nav2 path tracking after laser yaw flip
Two regressions introduced by f2dae1c (yaw flip of base_link->laser_link
static TF), addressed together since they share the same trigger.

A. App scan dots no longer matched walls
   - ros2_mobile_bridge._scan_to_points bypasses tf2 and was treating
     (px, py) as already in base_link. After the 180 deg static TF flip,
     points were rotated 180 deg vs the SLAM walls.
   - Add LASER_LINK_YAW_OFFSET = pi constant and compose
     yaw_eff = robot_yaw + LASER_LINK_YAW_OFFSET before rotating scan
     rays into map frame. Single source of truth aligns with the static
     TF; tf2 lookup deferred as future hygiene cleanup.
   - URDF laser_joint rpy reconciled (0 0 3.14159) so robot_state_
     publisher in visualization.launch.py won't contradict the live-SLAM
     launch.

B. Nav2 path tracking poor through curves
   - RPP min_lookahead_dist was 0.25 m, below the chassis R_min ~0.43 m
     (= wheelbase/tan(max_steer)). With velocity-scaled lookahead the
     carrot could land inside the smallest circle the car can draw,
     causing oscillation. Lifted to 0.45 (= R_min); lookahead_dist 0.45
     -> 0.55, max 0.70 -> 0.80.
   - regulated_linear_scaling_min_radius 0.45 -> 0.55 so the slowdown
     threshold sits above R_min — regulator decelerates BEFORE the
     chassis hits its physical turning limit, not at it.
   - planner_server motion_model_for_search REEDS_SHEPP -> DUBIN +
     RPP allow_reversing true -> false. Non-parking goals never need
     reverse; DUBIN paths never have cusps, eliminating the
     cusp-tracking error class. Parking mission node will dynamically
     re-enable REEDS_SHEPP + reversing per leg in phases 5-6 of
     docs/parking_plan.md.
   - controller_frequency 10 Hz -> 20 Hz so each tick is ~1.5 cm of
     travel instead of ~3 cm at 0.30 m/s. RPP is cheap; Pi5 has the
     headroom.

Joystick driving was always correct — it bypasses Nav2 — confirming
motors/wiring/polarity were fine and the issue was upstream in the
generation/following pipeline.

Co-Authored-By: Claude Opus 4.7 <noreply@anthropic.com>

File: src/parking_system/urdf/robot.urdf (robot description, URDF)
Before this commit: robot parking_robot, 3 links, 2 joints
Joints:
- joint laser_joint: origin xyz=0.15 0.0 0.12 rpy=0 0 0 -> xyz=0.15 0.0 0.12 rpy=0 0 3.14159

Commit message: Add direction-aware safety, snake fix, and 3-point park tuning
Test-driven V2 round addressing four still-broken symptoms:

- Wall stall (plan drawn but no motion near walls):
  * Disable RPP's internal collision check (use_collision_detection: false)
    so the controller no longer self-paralyzes when the chassis footprint
    overlaps wall inflation. Single collision authority is now the
    collision_monitor with the new direction-aware DirectionalStop.
  * Add DirectionalStop velocity_polygon with forward / reverse / stopped
    polygons. Reverse away from a wall is now allowed even though the
    forward polygon would see it - this is the wall-escape fix.
  * Inflation escape: relax to 0.0 m (was 0.02), hold for 10 s (was 6),
    remove plan-arrival early restore that re-inflated under the wheels
    mid-execution.

- Snake / oscillation on straight paths:
  * Push the carrot well outside the chassis footprint (min_lookahead
    0.20 -> 0.35, lookahead 0.22 -> 0.40, max 0.35 -> 0.55) and disable
    velocity-scaled lookahead so the carrot does not collapse to the
    floor at low cruise speed.
  * Disable use_cost_regulated_linear_velocity_scaling - in a 2x2 m
    testbed the chassis is always within inflation distance of
    something, so cost-ripple was the 2nd-largest snake contributor.
  * SMAC smoother w_smooth 0.3 -> 0.5, w_data 0.2 -> 0.1.
  * Bridge max_steer_rate 2.0 -> 1.5 rad/s, max_ax 0.5 -> 0.30,
    max_aw 0.7 -> 0.50; velocity_smoother caps tightened in lockstep.

- 180-degree reverse-park can't 3-point:
  * minimum_turning_radius 1.00 -> 0.85 m (testbed reality).
  * reverse_penalty 1.8 -> 1.2, change_penalty 0.5 -> 0.2 so the
    planner is willing to emit forward-reverse-forward sequences.
  * max_robot_pose_search_dist 3.0 -> 1.5 m so RPP doesn't re-latch
    onto the previous segment after a cusp.
  * Bridge cusp cooldown 250 -> 500 ms so the servo can fully swing
    at the lower 1.5 rad/s slew rate.
  * analytic_expansion_ratio 2.5 -> 2.0, max_planning_time 2 -> 4 s.

- Parking approach crashes / no clear deceleration:
  * approach_velocity_scaling_dist 0.60 -> 0.80 m,
    min_approach_linear_velocity 0.04 -> 0.03 m/s,
    xy_goal_tolerance 0.15 -> 0.10 m for precision.
  * DirectionalStop forward polygon is the new hard-stop before contact.

Robot dimensions sync (measured 27 cm L x 20 cm W):
- build_urdf.py chassis_length 0.30 -> 0.27.
- Static robot.urdf box 0.3 -> 0.27.
- local + global costmap footprints x +/-0.15 -> +/-0.135.
- DirectionalStop polygons rebuilt: forward [0.135, 0.235] x [+/-0.11],
  reverse [-0.235, -0.135] x [+/-0.11], stopped [+/-0.135] x [+/-0.10].

BT tweaks:
- RecoveryNode retries 6 -> 4, Wait 5 -> 2 s, BackUp 0.20/0.15 ->
  0.15/0.10 m so recovery doesn't drive into the opposite wall.

Co-Authored-By: Claude Opus 4.7 <noreply@anthropic.com>

File: src/parking_system/urdf/robot.urdf (robot description, URDF)
Before this commit: robot parking_robot, 3 links, 2 joints
Links:
- link base_link: geometry collision box size=0.27 0.2 0.1; visual box size=0.27 0.2 0.1

Commit message: Tune approach slowdown, planner bias, nav-bypass safety, SLAM drift
Two rounds of field-tuning bundled:

Round A — approach slowdown + creep escape + SLAM/URDF:
- RPP cruise 0.10->0.08 m/s, approach_velocity_scaling_dist 0.80->1.50 m,
  min_approach_linear_velocity 0.03->0.04. velocity_smoother cap
  0.12->0.10. Chassis reaches creep speed well before any wall.
- Inflation: local 0.08->0.10 m, global 0.10->0.12 m.
- DirectionalStop bumper 4->6 cm, min_points 8->5, linear_min/max
  +/-0.05 creep window so wall-adjacent poses can break out.
- nav2_pico_bridge max_vx_mps 0.30->0.15 (chassis never runs faster).
- URDF laser_joint yaw 3.14159->3.141593 (matches bridge math.pi).
- SLAM: loop_match response thresholds loosened 0.40/0.45->0.35/0.40,
  use_scan_barycenter off, scan_buffer_maximum_scan_distance 6.0.

Round B — planner tuning + path-active safety bypass:
- Planner: reverse_penalty 1.2->1.5, change_penalty 0.4->0.6 (operator
  reported reflexive cusps); smoother w_smooth 0.5->0.7, w_data
  0.1->0.05 (operator prefers longer, smoother paths).
- Path-active safety bypass: while a Nav2 goal is EXECUTING, the
  chassis follows /cmd_vel_smoothed (pre-collision_monitor) instead of
  /cmd_vel_safe, so a drawn path executes through what would otherwise
  be a hard-stop. nav2_pico_bridge gains a /cmd_vel_smoothed sub, a
  nav_bypass_active param (not persisted), and a 3-way arbiter
  (manual within window -> smoothed if bypass -> auto). ros2_mobile_
  bridge flips that param on Nav2 EXECUTING entry/exit and reports
  nav_bypass_active in /api/status + telemetry. Bridge clamps,
  200 ms watchdog, and Pico E-STOP latch remain the safety floor;
  operator E-STOP clears the bypass via the goal-cancel path.

Co-Authored-By: Claude Opus 4.7 (1M context) <noreply@anthropic.com>

File: src/parking_system/urdf/robot.urdf (robot description, URDF)
Before this commit: robot parking_robot, 3 links, 2 joints
Joints:
- joint laser_joint: origin xyz=0.01 0.0 0.07 rpy=0 0 3.14159 -> xyz=0.01 0.0 0.07 rpy=0 0 3.141593

File: src/parking_system/urdf/robot.urdf.xacro (robot description, xacro)
@@ -53,5 +53,5 @@
     <parent link="base_link"/>
     <child link="laser_link"/>
-    <origin xyz="{lidar_x} {lidar_y} {lidar_z}" rpy="0 0 3.14159"/>
+    <origin xyz="{lidar_x} {lidar_y} {lidar_z}" rpy="0 0 3.141593"/>
   </joint>
   <link name="camera_link">
